File: clawtronics/switches_etc.kicad_sch (KiCad schematic)
At the start: 7 parts, among them J6 Screw_Terminal_01x09, J7 Screw_Terminal_01x02, J8 Screw_Terminal_01x15, Q1 AO3400A

Commit message: figured out switches
Parts:
- added R26: 1K, Resistor_SMD:R_0603_1608Metric, symbol Device:R
- added R27: 660, Resistor_SMD:R_0603_1608Metric, symbol Device:R
- J6: footprint (none) -> TerminalBlock:TerminalBlock_MaiXu_MX126-5.0-09P_1x09_P5.00mm
- J7: renamed from J8; footprint (none) -> TerminalBlock:TerminalBlock_MaiXu_MX126-5.0-15P_1x15_P5.00mm
- J8: renamed from J7; footprint (none) -> TerminalBlock:TerminalBlock_MaiXu_MX126-5.0-02P_1x02_P5.00mm
- R28: renamed from R22; footprint (none) -> Resistor_SMD:R_0603_1608Metric
- R29: renamed from R23; footprint (none) -> Resistor_SMD:R_0603_1608Metric
Connections:
- net +5V: now also J7.9 (Pin_9), R26.1; no longer J6.1 (Pin_1), J6.3 (Pin_3), J6.5 (Pin_5), J6.9 (Pin_9)
- net GND: now also J7.10 (Pin_10), J7.11 (Pin_11), J7.2 (Pin_2), J7.3 (Pin_3), J7.4 (Pin_4), J7.5 (Pin_5), J7.6 (Pin_6), R27.2
- net GPIO45: now reaches J7.1 (Pin_1)
- net GPIO45: now also R26.2, R27.1
- net GNDPWR: now reaches J7.12 (Pin_12)
- net GNDPWR: now also J7.13 (Pin_13)
- net +24V: now reaches J7.14 (Pin_14)
- net +24V: now also J7.15 (Pin_15)
- net GPIO46: now reaches J7.7 (Pin_7)
- net GPIO47: now reaches J7.8 (Pin_8)
- new net GPIO11: J6.1 (Pin_1)
- new net GPIO12: J6.3 (Pin_3)
- new net GPIO13: J6.5 (Pin_5)
- new net GPIO17: J6.9 (Pin_9)
Other:
- note added: "AC/DC_IN+"
- note added: "AC/DC_IN-"
- note added: "EX_DOOR_OPEN"
- note added: "EX_PULSE_INHIBIT"
- note added: "GND"
- note added: "Internal 3.3V pullup"
- note added: "PULSE 1"
- note added: "PULSE 2"
- note added: "PULSE 3"
- note added: "PULSE 4"
- note added: "PULSE 5"
- note added: "PULSE 6"
- note added: "VCC"
